File: hardware/Power_v1/Power_module_v0.sch (KiCad schematic (older format))
At the start: 53 parts, among them J1 Conn_01x02, J2 Conn_02x03_motherboardconn, J3 USB_B_Micro, J4 Conn_01x02_battery, J5 Conn_01x06_programmer, J6 Conn_01x06_programmer, U1 BQ24040, U2 BQ25570, U3 TPS705, U4 PIC16F18446

Commit message: Power: renaming in schematic
Parts:
- S1, S2: symbol TPS22860:TPS22860 -> Power_module_v0-rescue:TPS22860-TPS22860
- U1: symbol BQ24040:BQ24040 -> Power_module_v0-rescue:BQ24040-BQ24040
- U3: symbol tps7a05:TPS705 -> Power_module_v0-rescue:TPS705-tps7a05
- U4: symbol PIC16F18446SSOP20pin:PIC16F18446 -> Power_module_v0-rescue:PIC16F18446-PIC16F18446SSOP20pin
- renumbered ROK3 to ROK1, ROK1 to ROK3, ROUT2 to ROUT1, ROUT1 to ROUT2, ROV2 to ROV1, ROV1 to ROV2
Other:
- note added: "BATT -> LDO -> 3V3"
- note added: "MPPT OK 80%"
- note added: "OK"
Changed lines of the file:
@@
 VSTOR
 $Comp
-L Device:R ROV1
+L Device:R ROV2
 U 1 1 5EDF021A
 P 3500 2450
-F 0 "ROV1" H 3570 2496 50  0000 L CNN
+F 0 "ROV2" H 3570 2496 50  0000 L CNN
 F 1 "7.32 M" H 3570 2405 50  0000 L CNN
 F 2 "Resistor_SMD:R_0805_2012Metric_Pad1.15x1.40mm_HandSolder" V 3430 2450 50  0001 C CNN
@@
 $EndComp
 $Comp
-L Device:R ROK1
+L Device:R ROK3
 U 1 1 5EDF088F
 P 3950 2450
-F 0 "ROK1" H 4020 2496 50  0000 L CNN
+F 0 "ROK3" H 4020 2496 50  0000 L CNN
 F 1 "1.9 M" H 4020 2405 50  0000 L CNN
 F 2 "Resistor_SMD:R_0805_2012Metric_Pad1.15x1.40mm_HandSolder" V 3880 2450 50  0001 C CNN
@@
 $EndComp
 $Comp
-L Device:R ROV2
+L Device:R ROV1
 U 1 1 5EDF0B8E
 P 3500 2850
-F 0 "ROV2" H 3570 2896 50  0000 L CNN
+F 0 "ROV1" H 3570 2896 50  0000 L CNN
 F 1 "5.61 M" H 3570 2805 50  0000 L CNN
 F 2 "Resistor_SMD:R_0805_2012Metric_Pad1.15x1.40mm_HandSolder" V 3430 2850 50  0001 C CNN
@@
 GND
 $Comp
-L Device:R ROK3
+L Device:R ROK1
 U 1 1 5EDF2C3E
 P 3950 3250
-F 0 "ROK3" H 4020 3296 50  0000 L CNN
+F 0 "ROK1" H 4020 3296 50  0000 L CNN
 F 1 "5.62M" H 4020 3205 50  0000 L CNN
 F 2 "Resistor_SMD:R_0805_2012Metric_Pad1.15x1.40mm_HandSolder" V 3880 3250 50  0001 C CNN
@@
 Connection ~ 3950 2300
 $Comp
-L Device:R ROUT1
+L Device:R ROUT2
 U 1 1 5EDF4059
 P 4600 2450
-F 0 "ROUT1" H 4670 2496 50  0000 L CNN
+F 0 "ROUT2" H 4670 2496 50  0000 L CNN
 F 1 "8.25 M" H 4670 2405 50  0000 L CNN
 F 2 "Resistor_SMD:R_0805_2012Metric_Pad1.15x1.40mm_HandSolder" V 4530 2450 50  0001 C CNN
@@
 $EndComp
 $Comp
-L Device:R ROUT2
+L Device:R ROUT1
 U 1 1 5EDF4212
 P 4600 2850
-F 0 "ROUT2" H 4670 2896 50  0000 L CNN
+F 0 "ROUT1" H 4670 2896 50  0000 L CNN
 F 1 "4.75 M" H 4670 2805 50  0000 L CNN
 F 2 "Resistor_SMD:R_0805_2012Metric_Pad1.15x1.40mm_HandSolder" V 4530 2850 50  0001 C CNN
@@
 	2900 1600 4150 1600
 $Comp
-L PIC16F18446SSOP20pin:PIC16F18446 U4
+L Power_module_v0-rescue:PIC16F18446-PIC16F18446SSOP20pin U4
 U 1 1 5EDFC64B
 P 8350 2600
@@
 3V3
 $Comp
-L TPS22860:TPS22860 S2
+L Power_module_v0-rescue:TPS22860-TPS22860 S2
 U 1 1 5EE49BD8
 P 5950 4000
@@
 $EndComp
 $Comp
-L TPS22860:TPS22860 S1
+L Power_module_v0-rescue:TPS22860-TPS22860 S1
 U 1 1 5EE4AA8C
 P 5900 5850
@@
 $EndComp
 $Comp
-L tps7a05:TPS705 U3
+L Power_module_v0-rescue:TPS705-tps7a05 U3
 U 1 1 5EEB36FB
 P 2550 6450
@@
 GND
 $Comp
-L BQ24040:BQ24040 U1
+L Power_module_v0-rescue:BQ24040-BQ24040 U1
 U 1 1 5EDFFF7A
 P 2050 4550
@@
 Text Notes 4950 4750 0    50   ~ 0
 8.2 k veranderen, zodat uw sampling ook tot aan 4.2V geraakt
+Text Notes 2200 6850 0    50   ~ 0
+BATT -> LDO -> 3V3
+Text Notes 4200 3450 0    50   ~ 0
+OK
+Text Notes 4250 3000 0    50   ~ 0
+OK
+Text Notes 4250 2600 0    50   ~ 0
+OK
+Text Notes 4950 2550 0    50   ~ 0
+OK
+Text Notes 4950 3000 0    50   ~ 0
+OK
+Text Notes 3300 3000 0    50   ~ 0
+OK
+Text Notes 3200 2500 0    50   ~ 0
+OK
+Text Notes 4600 1850 0    50   ~ 0
+OK
+Text Notes 3950 1150 0    50   ~ 0
+OK
+Text Notes 1400 1250 0    50   ~ 0
+OK
+Text Notes 1550 2750 0    50   ~ 0
+OK
+Text Notes 950  950  0    50   ~ 0
+MPPT OK 80%
 $EndSCHEMATC

Commit message: Power: HW notes
Other:
- note added: "X7R"
Changed lines of the file:
@@
 Text Notes 950  950  0    50   ~ 0
 MPPT OK 80%
+Text Notes 1150 2650 0    50   ~ 0
+X7R
 $EndSCHEMATC

Commit message: Power: HW buck layout
Parts:
- J3: symbol Connector:USB_B_Micro -> Power_module_v0-rescue:USB_B_Micro-Connector
Changed lines of the file:
@@
 USB charger IC
 $Comp
-L Connector:USB_B_Micro J3
+L Power_module_v0-rescue:USB_B_Micro-Connector J3
 U 1 1 5EE0210B
 P 10100 3050
