File: hardware/Power_v3/kicadproject/Power_module_v1.sch (KiCad schematic (older format))
At the start: 64 parts, among them J1 Conn_01x02, J2 Conn_02x03_motherboardconn, J3 USB_B_Micro, J4 Conn_01x02_battery, J5 Conn_01x06_programmer, J6 Conn_01x06_programmer, U1 BQ24040, U2 BQ25570, U3 TPS705, U4 PIC16F18446

Commit message: Power: conversion config + maybe change in hw
Other:
- note added: "ROK3 1.258M 1.27M\nROK2 6.668M 6.81M\nROK1 5.074M 5.11M"
Changed lines of the file:
@@
 	1    0    0    -1
 $EndComp
+Text Notes 4100 3700 0    50   ~ 0
+ROK3   1.258M   1.27M\nROK2   6.668M   6.81M\nROK1   5.074M   5.11M
 $EndSCHEMATC
