File: hardware/Power_v4/kicadproject/Power_module_v1.sch (KiCad schematic (older format))
At the start: 64 parts, among them J1 Conn_01x02, J2 Conn_02x03_motherboardconn, J3 USB_B_Micro, J4 Conn_01x02_battery, J5 Conn_01x06_programmer, J6 Conn_01x06_programmer, U1 BQ24040, U2 BQ25570, U3 TPS705, U4 PIC16F18446

Commit message: Update hardware schematics
Parts:
- R7: value 27k -> 4k7
Changed lines of the file:
@@
 P 5100 6650
 F 0 "R7" H 5170 6696 50  0000 L CNN
-F 1 "27k" H 5170 6605 50  0000 L CNN
+F 1 "4k7" H 5170 6605 50  0000 L CNN
 F 2 "Resistor_SMD:R_0805_2012Metric_Pad1.15x1.40mm_HandSolder" V 5030 6650 50  0001 C CNN
 F 3 "~" H 5100 6650 50  0001 C CNN
