File: hardware/Buttons/kicadproject/STEM.sch (KiCad schematic (older format))
At the start: 23 parts, among them IC1 PIC16F18446-I_SS, J1 PICKit3, J2 MASTER

Commit message: Update Sensor Module
Parts:
- removed S1, S2, S3, S4: 3006.2114, TactileSwitchLed_30062114_footprint:30062114, symbol TactileSwitchLed_3006.2114:3006.2114
- added U1, U2, U3, U4: button, Button_Ali:aliButton, symbol Button_Ali:button
- C1, C2, C3, C4, C5: footprint Capacitor_SMD:C_0805_2012Metric_Pad1.15x1.40mm_HandSolder -> Capacitor_SMD:C_0805_2012Metric_Pad1.18x1.45mm_HandSolder
- IC1: symbol PIC16f18446:PIC16F18446-I_SS -> STEM-rescue:PIC16F18446-I_SS-PIC16f18446
- LED1: symbol LED_SML-D12Y1WT86:SML-D12Y1WT86 -> STEM-rescue:SML-D12Y1WT86-LED_SML-D12Y1WT86
- R1, R10, R2, R3, R4, R9: footprint Resistor_SMD:R_0805_2012Metric_Pad1.15x1.40mm_HandSolder -> Resistor_SMD:R_0805_2012Metric_Pad1.20x1.40mm_HandSolder
- R5, R7: value 1k -> 100k; footprint Resistor_SMD:R_0805_2012Metric_Pad1.15x1.40mm_HandSolder -> Resistor_SMD:R_0805_2012Metric_Pad1.20x1.40mm_HandSolder
- R6, R8: value 100k -> 1k; footprint Resistor_SMD:R_0805_2012Metric_Pad1.15x1.40mm_HandSolder -> Resistor_SMD:R_0805_2012Metric_Pad1.20x1.40mm_HandSolder
Connections:
- wire segments 94 -> 152
Other:
- moved on the sheet: C2, R2, R3
